Commit message: replay episode blender version code updated

File: assets/shelf/shelf_for_blender_backup.urdf (robot description, URDF)
Before this commit: robot plane, 6 links, 5 joints
Links:
- link shelf_back: geometry collision mesh filename=meshes/shelf_back.obj; visual mesh filename=meshes/shelf_back.obj
- link shelf_bottom: geometry collision mesh filename=meshes/shelf_bottom.obj; visual mesh filename=meshes/shelf_bottom.obj
- link shelf_left: geometry collision mesh filename=meshes/shelf_left.obj; visual mesh filename=meshes/shelf_left.obj
- link shelf_middle: geometry collision mesh filename=meshes/shelf_middle.obj; visual mesh filename=meshes/shelf_middle.obj
- link shelf_right: geometry collision mesh filename=meshes/shelf_right.obj; visual mesh filename=meshes/shelf_right.obj
- link shelf_upper: geometry collision mesh filename=meshes/shelf_upper.obj; visual mesh filename=meshes/shelf_upper.obj
